File: sidi-base.brd (EAGLE design)
At the start: 58.1 x 69.8 mm, 22 parts, among them IC1 ATMEGA168-20P, Q1 16mhz

Commit message: Oops
Connections:
- net GND: no longer R1.1
- net VCC: now also R1.1
Routing:
- net VCC: track 164.2 -> 166.8 mm
Changed lines of the file:
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@@
 </signal>
 <signal name="GND">
-<contactref element="R1" pad="1"/>
-<contactref element="S1" pad="4"/>
-<contactref element="S1" pad="3"/>
 <contactref element="POWER" pad="2"/>
 <contactref element="LED1" pad="K"/>
@@
 </polygon>
 <contactref element="C3" pad="2"/>
+<contactref element="S1" pad="4"/>
+<contactref element="S1" pad="3"/>
 </signal>
 <signal name="VCC">
@@
 <wire x1="45.72" y1="33.02" x2="43.18" y2="33.02" width="0.4064" layer="1"/>
 <wire x1="46.99" y1="62.23" x2="43.18" y2="66.04" width="0.6096" layer="1"/>
-<wire x1="43.18" y1="66.04" x2="11.43" y2="66.04" width="0.6096" layer="1"/>
+<wire x1="43.18" y1="66.04" x2="34.29" y2="66.04" width="0.6096" layer="1"/>
+<wire x1="34.29" y1="66.04" x2="11.43" y2="66.04" width="0.6096" layer="1"/>
 <wire x1="11.43" y1="66.04" x2="10.16" y2="64.77" width="0.6096" layer="1"/>
 <wire x1="49.53" y1="64.77" x2="48.26" y2="66.04" width="0.6096" layer="1"/>
 <wire x1="48.26" y1="66.04" x2="43.18" y2="66.04" width="0.6096" layer="1"/>
 <wire x1="8.89" y1="35.56" x2="8.89" y2="40.64" width="0.6096" layer="1"/>
+<contactref element="R1" pad="1"/>
+<wire x1="34.29" y1="63.5" x2="34.29" y2="66.04" width="0.4064" layer="1"/>
 </signal>
 <signal name="N$5">
