File: sidi-base.brd (EAGLE design)
At the start: 58.1 x 69.8 mm, 22 parts, among them IC1 ATMEGA168-20P, Q1 16mhz

Commit message: Latest revision to the board. Control surface code silenced.
Parts:
- removed D1: 1N4148DO35-7, diode:DO35-7
- added D2: (no value), adafruit:DO-1N4148
- added R8: 10k, resistor:0207/7
- R7: value 330ohm -> 470ohm
- moved R7 6.35 mm to (12.7, 47.0)
- moved R6 4.58 mm to (12.7, 24.1)
- moved OK1 2.54 mm to (12.7, 34.3)
- moved LED1 1.80 mm to (8.89, 52.1)
- moved R4 1.80 mm to (12.7, 57.1)
- moved C1 1.27 mm to (24.1, 35.6)
- moved C2 1.27 mm to (24.1, 25.4)
- moved Q1 1.27 mm to (30.5, 30.5)
Connections:
- new net N$1: OK1.7, R8.1
- net GND: now also R8.2; no longer R1.1
- net N$18: now also D2.A; no longer D1.A
- net N$20: now also D2.C; no longer D1.C
- net VCC: now also R1.1
Routing:
- net N$1: track 0.00 -> 5.08 mm
- net N$19: track 4.56 -> 8.00 mm
- net N$7: track 13.9 -> 17.1 mm
- net N$6: track 12.8 -> 16.0 mm
- net VCC: track 164.2 -> 166.5 mm
- net N$18: track 20.3 -> 21.8 mm
- net N$23: track 31.5 -> 32.7 mm
- net N$20: track 8.67 -> 8.15 mm
Other:
- board text added: "1"
- board text added: "ONESIDDY REV 2"
- board text added: "ONESIDDY REV 2 BASE BOARD"
- board text removed: "ONESIDDY REV 1"
- board text removed: "ONESIDDY REV 1 BASE BOARD"
