File: sidi-base.sch (EAGLE design)
At the start: 22 parts, among them IC1 ATMEGA168-20P, Q1 16mhz

Commit message: Latest revision to the board. Control surface code silenced.
Parts:
- removed D1: 1N4148DO35-7, diode:1N4148DO35-7
- added D2: (no value), adafruit:DIODEDO-1N4148
- added R8: 10k, resistor:R-EU_0207/7
- R7: value 330ohm -> 470ohm
Connections:
- new net N$1: OK1.VB, R8.1
- net GND: now also R8.2; no longer R1.1
- net N$18: now also D2.A; no longer D1.A
- net N$20: now also D2.C; no longer D1.C
- net VCC: now also R1.1
Other:
- moved on the sheet: R7
